Commit message: Nuevas poses, de mesa a cocina

File: ktmpb/ktmpb_interfaces/demos/models/obstacles/kitchen/restaurant_table.urdf (robot description, URDF)
Before this commit: robot mesa_simple2, 1 links, 0 joints
Links:
- link base: geometry collision mesh filename=final_project_models/outdoor_kitchen.dae.dae scale=1 1 1; visual mesh filename=final_project_models/outdoor_kitchen.dae.dae scale=1 1 1
