Commit message: works fine (aparte de 2 colisiones xd)

File: ktmpb/ktmpb_interfaces/demos/models/obstacles/kitchen/can_1.urdf (robot description, URDF)
Before this commit: robot can_1, 1 links, 0 joints
Links:
- link base: geometry collision cylinder length=0.07 radius=0.025; visual cylinder length=0.07 radius=0.025

File: ktmpb/ktmpb_interfaces/demos/models/obstacles/kitchen/can_1_small.urdf (robot description, URDF)
Before this commit: robot can_1_small, 1 links, 0 joints
Links:
- link base: geometry collision mesh filename=can/cokecan.dae scale=0.0254 0.0254 0.0254; visual mesh filename=can/cokecan2.dae scale=0.0254 0.0254 0.0254

File: ktmpb/ktmpb_interfaces/demos/models/obstacles/kitchen/can_2.urdf (robot description, URDF)
Before this commit: robot can_2, 1 links, 0 joints
Links:
- link base: geometry collision cylinder length=0.07 radius=0.025; visual cylinder length=0.07 radius=0.025

File: ktmpb/ktmpb_interfaces/demos/models/obstacles/kitchen/can_3.urdf (robot description, URDF)
Before this commit: robot can_3, 1 links, 0 joints
Links:
- link base: geometry collision cylinder length=0.07 radius=0.025; visual cylinder length=0.07 radius=0.025
