Commit message: este programa me va a volver loco

File: ktmpb/ktmpb_interfaces/demos/models/robots/ur3_robotniq_A.urdf (robot description, URDF)
Before this commit: robot ur3_robotniq_A, 21 links, 20 joints
Links:
- link gripper_left_coupler: geometry collision box size=0.00 0.0 0.00; visual mesh filename=robotiq/visual/coupler.dae scale=0.001 0.001 0.001
- link gripper_right_coupler: geometry collision box size=0.00 0.0 0.00; visual mesh filename=robotiq/visual/coupler.dae scale=0.001 0.001 0.001
